File: flex/flex.kicad_sch (KiCad schematic)
At the start: 11 parts, among them SW1 SW_Push, SW2 SW_Push, SW3 SW_Push

Commit message: blend
Connections:
- net DISP_T_IRQ: now also A1.11 (GPIO8); no longer A1.6 (GPIO4)
- net SD_MISO: now also A1.6 (GPIO4); no longer A1.11 (GPIO8)
Changed lines of the file:
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@@
 	)
 	(label "DISP_T_IRQ"
-		(at 105.41 93.98 0)
+		(at 105.41 104.14 0)
 		(effects
 			(font
@@
 	)
 	(label "SD_MISO"
-		(at 105.41 104.14 0)
+		(at 105.41 93.98 0)
 		(effects
 			(font
@@
 		)
 		(pin "6"
+			(alternate "SPI0_RX")
 		)
 		(pin "18"
@@
 		)
 		(pin "11"
-			(alternate "SPI1_RX")
 		)
 		(pin "2"
